Commit message: innovation fair code

File: src/turtlebot3/turtlebot3_description/urdf/turtlebot3_burger.urdf (robot description, URDF)
Before this commit: robot turtlebot3_burger, 7 links, 6 joints
Links:
- added link camera_link, mass 0.03; collision box size=0.025 0.024 0.009; visual box size=0.025 0.024 0.009
- added link camera_optical_frame
Joints:
- added joint camera_joint: type fixed, parent base_link, child camera_link, origin xyz=0.05 0 0.10 rpy=0 -0.26 0
- added joint camera_optical_joint: type fixed, parent camera_link, child camera_optical_frame, origin xyz=0 0 0 rpy=-1.5708 0 -1.5708
